File: design/lna.kicad_sch (KiCad schematic)
At the start: 22 parts, among them J5 SMA, U9 ADA4930-1

Commit message: Added FTDI layout
Parts:
- TP1, TP2, TP3: footprint TestPoint:TestPoint_Loop_D2.50mm_Drill1.0mm_LowProfile -> TestPoint:TestPoint_Pad_D1.0mm
Changed lines of the file:
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@@
-(kicad_sch (version 20200506) (host eeschema "5.99.0-unknown-acdfeee~101~ubuntu18.04.1")
+(kicad_sch (version 20200506) (host eeschema "5.99.0-unknown-c3b50d3~101~ubuntu18.04.1")
   (page "A4")
   (title_block
@@
     (property "Reference" "TP1" (id 0) (at 83.693 56.134 90))
     (property "Value" "TestPoint_Probe" (id 1) (at 83.693 58.4454 90))
-    (property "Footprint" "TestPoint:TestPoint_Loop_D2.50mm_Drill1.0mm_LowProfile" (id 2) (at 85.09 58.42 0)
+    (property "Footprint" "TestPoint:TestPoint_Pad_D1.0mm" (id 2) (at 85.09 58.42 0)
       (effects (font (size 1.27 1.27)) hide)
     )
@@
     (property "Reference" "TP2" (id 0) (at 214.503 82.804 90))
     (property "Value" "TestPoint_Probe" (id 1) (at 214.503 85.1154 90))
-    (property "Footprint" "TestPoint:TestPoint_Loop_D2.50mm_Drill1.0mm_LowProfile" (id 2) (at 215.9 85.09 0)
+    (property "Footprint" "TestPoint:TestPoint_Pad_D1.0mm" (id 2) (at 215.9 85.09 0)
       (effects (font (size 1.27 1.27)) hide)
     )
@@
     (property "Reference" "TP3" (id 0) (at 214.503 105.3338 0))
     (property "Value" "TestPoint_Probe" (id 1) (at 214.503 107.6452 0))
-    (property "Footprint" "TestPoint:TestPoint_Loop_D2.50mm_Drill1.0mm_LowProfile" (id 2) (at 210.82 100.33 0)
-      (effects (font (size 1.27 1.27)) hide)
-    )
+    (property "Footprint" "TestPoint:TestPoint_Pad_D1.0mm" (id 2) (at 210.82 100.33 0)
+      (effects (font (size 1.27 1.27)) hide)
+    )
