File: design/digitizer_fpga_10b_100MSPS.kicad_sch (KiCad schematic)
At the start: 13 parts

Commit message: Updated schematic
Parts:
- gave numbers to parts that had none: 8
Changed lines of the file:
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@@
   )
   (symbol (lib_id "KLIB_Mechanical:Fiducial") (at 118.11 170.18 0) (unit 1)
-    (property "Reference" "FD?" (id 0) (at 121.92 168.91 0)
+    (property "Reference" "FD1" (id 0) (at 121.92 168.91 0)
       (effects (font (size 1.27 1.27)) (justify left))
     )
@@
   )
   (symbol (lib_id "KLIB_Mechanical:Fiducial") (at 118.11 176.53 0) (unit 1)
-    (property "Reference" "FD?" (id 0) (at 121.92 175.26 0)
+    (property "Reference" "FD2" (id 0) (at 121.92 175.26 0)
       (effects (font (size 1.27 1.27)) (justify left))
     )
@@
   )
   (symbol (lib_id "KLIB_Mechanical:Fiducial") (at 118.11 184.15 0) (unit 1)
-    (property "Reference" "FD?" (id 0) (at 121.92 182.88 0)
+    (property "Reference" "FD3" (id 0) (at 121.92 182.88 0)
       (effects (font (size 1.27 1.27)) (justify left))
     )
@@
   )
   (symbol (lib_id "KLIB_Mechanical:Fiducial") (at 118.11 190.5 0) (unit 1)
-    (property "Reference" "FD?" (id 0) (at 121.92 189.23 0)
+    (property "Reference" "FD4" (id 0) (at 121.92 189.23 0)
       (effects (font (size 1.27 1.27)) (justify left))
     )
@@
   )
   (symbol (lib_id "KLIB_Mechanical:Fiducial") (at 143.51 170.18 0) (unit 1)
-    (property "Reference" "FD?" (id 0) (at 147.32 168.91 0)
+    (property "Reference" "FD5" (id 0) (at 147.32 168.91 0)
       (effects (font (size 1.27 1.27)) (justify left))
     )
@@
   )
   (symbol (lib_id "KLIB_Mechanical:Fiducial") (at 143.51 176.53 0) (unit 1)
-    (property "Reference" "FD?" (id 0) (at 147.32 175.26 0)
+    (property "Reference" "FD6" (id 0) (at 147.32 175.26 0)
       (effects (font (size 1.27 1.27)) (justify left))
     )
@@
   )
   (symbol (lib_id "KLIB_Mechanical:Fiducial") (at 143.51 184.15 0) (unit 1)
-    (property "Reference" "FD?" (id 0) (at 147.32 182.88 0)
+    (property "Reference" "FD7" (id 0) (at 147.32 182.88 0)
       (effects (font (size 1.27 1.27)) (justify left))
     )
@@
   )
   (symbol (lib_id "KLIB_Mechanical:Fiducial") (at 143.51 190.5 0) (unit 1)
-    (property "Reference" "FD?" (id 0) (at 147.32 189.23 0)
+    (property "Reference" "FD8" (id 0) (at 147.32 189.23 0)
       (effects (font (size 1.27 1.27)) (justify left))
     )
@@
     (path "/6c07a7e5-f136-44bb-8086-ba05ad45ce64" (reference "#PWR03") (unit 1))
     (path "/f54593db-a2df-44c5-8513-2bde6eaa3b94" (reference "#PWR04") (unit 1))
-    (path "/15990d51-6613-410a-b9bf-b9c16c73e9f4" (reference "FD?") (unit 1))
-    (path "/2b79b4d8-433b-425e-b209-129ffcd949fd" (reference "FD?") (unit 1))
-    (path "/9c9d4db9-f696-4d68-a52a-db12895f4bea" (reference "FD?") (unit 1))
-    (path "/a09b0666-8d86-4dae-b667-dcbb3a29bf60" (reference "FD?") (unit 1))
-    (path "/bd0b34e1-8137-46a6-a773-b5659f7ffad2" (reference "FD?") (unit 1))
-    (path "/cc908382-2291-421b-aa1a-d790d0402769" (reference "FD?") (unit 1))
-    (path "/e31f8e3b-dd48-40c1-b5d6-3b89aa06f3bc" (reference "FD?") (unit 1))
-    (path "/f1b3ec91-2292-4d03-b160-728826e2eac1" (reference "FD?") (unit 1))
+    (path "/cc908382-2291-421b-aa1a-d790d0402769" (reference "FD1") (unit 1))
+    (path "/f1b3ec91-2292-4d03-b160-728826e2eac1" (reference "FD2") (unit 1))
+    (path "/2b79b4d8-433b-425e-b209-129ffcd949fd" (reference "FD3") (unit 1))
+    (path "/e31f8e3b-dd48-40c1-b5d6-3b89aa06f3bc" (reference "FD4") (unit 1))
+    (path "/15990d51-6613-410a-b9bf-b9c16c73e9f4" (reference "FD5") (unit 1))
+    (path "/a09b0666-8d86-4dae-b667-dcbb3a29bf60" (reference "FD6") (unit 1))
+    (path "/9c9d4db9-f696-4d68-a52a-db12895f4bea" (reference "FD7") (unit 1))
+    (path "/bd0b34e1-8137-46a6-a773-b5659f7ffad2" (reference "FD8") (unit 1))
     (path "/0986990b-68f7-46ae-983b-508b0be78074" (reference "GR1") (unit 1))
     (path "/f56eaa1e-ba52-456d-99dd-e4fffeedc129" (reference "H1") (unit 1))

Commit message: Updated notes
Other:
- note added: "+1V0"
- note added: "+1V8"
- note added: "+3V3A"
- note added: "+3V3D"
Changed lines of the file:
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@@
-(kicad_sch (version 20200512) (host eeschema "5.99.0-unknown-598ed8b~101~ubuntu18.04.1")
-  (page 1 8)
+(kicad_sch (version 20200608) (host eeschema "5.99.0-unknown-ad69e44~101~ubuntu18.04.1")
+  (page 9 8)
   (paper "A4")
   (title_block
@@
   )
   (polyline (pts (xy 120.65 102.87) (xy 121.92 102.87))
-    (stroke (width 0.1524) (type dash) (color 0 0 0 0))
+    (stroke (width 0.1524) (type solid) (color 0 0 0 0))
   )
   (polyline (pts (xy 121.92 100.33) (xy 125.73 102.87))
-    (stroke (width 0.1524) (type dash) (color 0 0 0 0))
+    (stroke (width 0.1524) (type solid) (color 0 0 0 0))
   )
   (polyline (pts (xy 121.92 105.41) (xy 121.92 100.33))
-    (stroke (width 0.1524) (type dash) (color 0 0 0 0))
+    (stroke (width 0.1524) (type solid) (color 0 0 0 0))
   )
   (polyline (pts (xy 121.92 105.41) (xy 125.73 102.87))
-    (stroke (width 0.1524) (type dash) (color 0 0 0 0))
+    (stroke (width 0.1524) (type solid) (color 0 0 0 0))
   )
   (polyline (pts (xy 125.73 102.87) (xy 127 102.87))
-    (stroke (width 0.1524) (type dash) (color 0 0 0 0))
-  )
-  (symbol (lib_id "KLIB_Power:GND") (at 16.51 190.5 0) (unit 1)
+    (stroke (width 0.1524) (type solid) (color 0 0 0 0))
+  )
+  (text "+3V3A" (at 114.3 60.96 180)
+    (effects (font (size 1.27 1.27)) (justify right bottom))
+  )
+  (text "+3V3D" (at 137.16 60.96 180)
+    (effects (font (size 1.27 1.27)) (justify right bottom))
+  )
+  (text "+1V8" (at 160.02 60.96 180)
+    (effects (font (size 1.27 1.27)) (justify right bottom))
+  )
+  (text "+1V0" (at 185.42 60.96 180)
+    (effects (font (size 1.27 1.27)) (justify right bottom))
+  )
+  (symbol (lib_id "KLIB_Power:GND") (at 16.51 190.5 0)
+    (in_bom yes) (on_board yes)
     (property "Reference" "#PWR01" (id 0) (at 16.51 195.58 0)
       (effects (font (size 1.27 1.27)) hide)
@@
     )
   )
-  (symbol (lib_id "KLIB_Power:GND") (at 35.56 190.5 0) (unit 1)
+  (symbol (lib_id "KLIB_Power:GND") (at 35.56 190.5 0)
+    (in_bom yes) (on_board yes)
     (property "Reference" "#PWR02" (id 0) (at 35.56 195.58 0)
       (effects (font (size 1.27 1.27)) hide)
@@
     )
   )
-  (symbol (lib_id "KLIB_Power:GND") (at 54.61 190.5 0) (unit 1)
+  (symbol (lib_id "KLIB_Power:GND") (at 54.61 190.5 0)
+    (in_bom yes) (on_board yes)
     (property "Reference" "#PWR03" (id 0) (at 54.61 195.58 0)
       (effects (font (size 1.27 1.27)) hide)
@@
     )
   )
-  (symbol (lib_id "KLIB_Power:GND") (at 73.66 190.5 0) (unit 1)
+  (symbol (lib_id "KLIB_Power:GND") (at 73.66 190.5 0)
+    (in_bom yes) (on_board yes)
     (property "Reference" "#PWR04" (id 0) (at 73.66 195.58 0)
       (effects (font (size 1.27 1.27)) hide)
@@
     )
   )
-  (symbol (lib_id "KLIB_Mechanical:Fiducial") (at 118.11 170.18 0) (unit 1)
+  (symbol (lib_id "KLIB_Mechanical:Fiducial") (at 118.11 170.18 0)
+    (in_bom yes) (on_board yes)
     (property "Reference" "FD1" (id 0) (at 121.92 168.91 0)
       (effects (font (size 1.27 1.27)) (justify left))
@@
     )
   )
-  (symbol (lib_id "KLIB_Mechanical:Fiducial") (at 118.11 176.53 0) (unit 1)
+  (symbol (lib_id "KLIB_Mechanical:Fiducial") (at 118.11 176.53 0)
+    (in_bom yes) (on_board yes)
     (property "Reference" "FD2" (id 0) (at 121.92 175.26 0)
       (effects (font (size 1.27 1.27)) (justify left))
@@
     )
   )
-  (symbol (lib_id "KLIB_Mechanical:Fiducial") (at 118.11 184.15 0) (unit 1)
+  (symbol (lib_id "KLIB_Mechanical:Fiducial") (at 118.11 184.15 0)
+    (in_bom yes) (on_board yes)
     (property "Reference" "FD3" (id 0) (at 121.92 182.88 0)
       (effects (font (size 1.27 1.27)) (justify left))
@@
     )
   )
-  (symbol (lib_id "KLIB_Mechanical:Fiducial") (at 118.11 190.5 0) (unit 1)
+  (symbol (lib_id "KLIB_Mechanical:Fiducial") (at 118.11 190.5 0)
+    (in_bom yes) (on_board yes)
     (property "Reference" "FD4" (id 0) (at 121.92 189.23 0)
       (effects (font (size 1.27 1.27)) (justify left))
@@
     )
   )
-  (symbol (lib_id "KLIB_Mechanical:Fiducial") (at 143.51 170.18 0) (unit 1)
+  (symbol (lib_id "KLIB_Mechanical:Fiducial") (at 143.51 170.18 0)
+    (in_bom yes) (on_board yes)
     (property "Reference" "FD5" (id 0) (at 147.32 168.91 0)
       (effects (font (size 1.27 1.27)) (justify left))
@@
     )
   )
-  (symbol (lib_id "KLIB_Mechanical:Fiducial") (at 143.51 176.53 0) (unit 1)
+  (symbol (lib_id "KLIB_Mechanical:Fiducial") (at 143.51 176.53 0)
+    (in_bom yes) (on_board yes)
     (property "Reference" "FD6" (id 0) (at 147.32 175.26 0)
       (effects (font (size 1.27 1.27)) (justify left))
@@
     )
   )
-  (symbol (lib_id "KLIB_Mechanical:Fiducial") (at 143.51 184.15 0) (unit 1)
+  (symbol (lib_id "KLIB_Mechanical:Fiducial") (at 143.51 184.15 0)
+    (in_bom yes) (on_board yes)
     (property "Reference" "FD7" (id 0) (at 147.32 182.88 0)
       (effects (font (size 1.27 1.27)) (justify left))
@@
     )
   )
-  (symbol (lib_id "KLIB_Mechanical:Fiducial") (at 143.51 190.5 0) (unit 1)
+  (symbol (lib_id "KLIB_Mechanical:Fiducial") (at 143.51 190.5 0)
+    (in_bom yes) (on_board yes)
     (property "Reference" "FD8" (id 0) (at 147.32 189.23 0)
       (effects (font (size 1.27 1.27)) (justify left))
@@
     )
   )
-  (symbol (lib_id "KLIB_Mechanical:Bolt_Pad") (at 16.51 190.5 0) (unit 1)
+  (symbol (lib_id "KLIB_Mechanical:Bolt_Pad") (at 16.51 190.5 0)
+    (in_bom yes) (on_board yes)
     (property "Reference" "H1" (id 0) (at 21.59 186.69 0)
       (effects (font (size 1.27 1.27)) (justify left))
@@
     )
   )
-  (symbol (lib_id "KLIB_Mechanical:Bolt_Pad") (at 35.56 190.5 0) (unit 1)
+  (symbol (lib_id "KLIB_Mechanical:Bolt_Pad") (at 35.56 190.5 0)
+    (in_bom yes) (on_board yes)
     (property "Reference" "H2" (id 0) (at 40.64 186.69 0)
       (effects (font (size 1.27 1.27)) (justify left))
@@
     )
   )
-  (symbol (lib_id "KLIB_Mechanical:Bolt_Pad") (at 54.61 190.5 0) (unit 1)
+  (symbol (lib_id "KLIB_Mechanical:Bolt_Pad") (at 54.61 190.5 0)
+    (in_bom yes) (on_board yes)
     (property "Reference" "H3" (id 0) (at 59.69 186.69 0)
       (effects (font (size 1.27 1.27)) (justify left))
@@
     )
   )
-  (symbol (lib_id "KLIB_Mechanical:Bolt_Pad") (at 73.66 190.5 0) (unit 1)
+  (symbol (lib_id "KLIB_Mechanical:Bolt_Pad") (at 73.66 190.5 0)
+    (in_bom yes) (on_board yes)
     (property "Reference" "H4" (id 0) (at 78.74 186.69 0)
       (effects (font (size 1.27 1.27)) (justify left))
@@
     )
   )
-  (symbol (lib_id "KLIB_Logo:Wykys") (at 271.78 173.99 0) (unit 1)
+  (symbol (lib_id "KLIB_Logo:Wykys") (at 271.78 173.99 0)
+    (in_bom yes) (on_board yes)
     (property "Reference" "GR1" (id 0) (at 271.78 177.4444 0)
       (effects (font (size 1.27 1.27)) hide)

Commit message: Added net classes
Other:
- title: Digitizer 10b 105 MSPS with FPGA -> Digitizer 10b 100 MSPS with FPGA
Changed lines of the file:
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@@
-(kicad_sch (version 20200618) (host eeschema "5.99.0-unknown-f420396~101~ubuntu18.04.1")
+(kicad_sch (version 20200714) (host eeschema "5.99.0-unknown-039b6fd~102~ubuntu18.04.1")
   (page 1 8)
   (paper "A4")
   (title_block
-    (title "Digitizer 10b 105 MSPS with FPGA")
+    (title "Digitizer 10b 100 MSPS with FPGA")
     (date "2020-03-09")
     (rev "1.0")
